File: hardware/pcb/argokey.kicad_pcb (KiCad board)
At the start: 2 copper layers, 173 parts, among them J1 USB_BOOT, J2 GPIO, J3 Screen, J4 Debug, U1 W25Q128JVS, U2 RP2040, U3 NCP1117-3.3_SOT223

Commit message: PCB: Most traces
Parts:
- added J5: USB_C, Connector_USB:USB_C_Receptacle_Amphenol_12401548E4-2A, F.Cu at (70.8, 91.1)
- added SW1: RotaryEnc, Rotary_Encoder:RotaryEncoder_Alps_EC12E-Switch_Vertical_H20mm, F.Cu at (69.0, 106.9)
- added SW2: RESET, Button_Switch_THT:SW_PUSH_6mm_H4.3mm, F.Cu at (61.2, 88.4)
- added Y1: ABLS-12.000MHZ-B4-T, RP2040_minimal:Crystal_SMD_HC49-US, F.Cu at (79.8, 157.8)
- C1, C2, J2, J4, R1, R2, R6: moved to B.Cu
- U2: footprint RP2040:RP2040 -> RP2040_minimal:RP2040-QFN-56
- moved C1 104.4 mm to (61.9, 107.0), turned to 180 degrees
- moved R6 102.8 mm to (68.2, 92.3)
- moved R7 102.8 mm to (73.5, 98.2), turned to 180 degrees
- moved C2 102.3 mm to (61.9, 111.7)
- moved R9 101.8 mm to (71.7, 98.8), turned to 90 degrees
- moved R10 98.4 mm to (69.9, 98.8), turned to 90 degrees
- moved R1 95.1 mm to (61.9, 102.8), turned to 180 degrees
- moved R8 95.0 mm to (73.9, 156.9), turned to 180 degrees
- moved R5 91.8 mm to (72.5, 151.4), turned to -135 degrees
- moved C18 90.9 mm to (50.6, 120.0)
- moved R2 83.7 mm to (61.9, 115.9), turned to 180 degrees
- moved C15 75.8 mm to (39.9, 114.0), turned to 90 degrees
- moved R4 73.0 mm to (41.2, 166.4), turned to 135 degrees
- moved C14 70.8 mm to (76.4, 156.1), turned to -90 degrees
- moved C16 64.9 mm to (73.6, 154.2)
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Connections:
- S13 pad 1: Col 2 -> Col 1
- S18 pad 1: Col 3 -> Col 2
- S23 pad 1: Col 4 -> Col 3
Routing:
- net Col 9: track 0.00 -> 414.4 mm
- net Col 8: track 0.00 -> 392.4 mm
- net Col 11: track 0.00 -> 390.2 mm
- net Col 10: track 0.00 -> 365.6 mm
- net Col 12: track 0.00 -> 359.5 mm
- net Col 13: track 0.00 -> 356.5 mm
- net Row 4: track 0.00 -> 336.5 mm
- net Row 2: track 0.00 -> 331.8 mm
- net Row 3: track 0.00 -> 317.2 mm
- net Col 6: track 0.00 -> 316.9 mm
- net Row 1: track 0.00 -> 280.0 mm
- net Row 0: track 0.00 -> 277.9 mm
- net Col 5: track 0.00 -> 235.9 mm
- net Col 4: track 0.00 -> 201.5 mm
- net Col 3: track 0.00 -> 185.0 mm
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
Commit message: PCB: Most traces
Parts:
- D9, R7: moved to B.Cu
- J2: footprint Connector_PinHeader_2.54mm:PinHeader_1x12_P2.54mm_Horizontal -> Connector_PinSocket_2.54mm:PinSocket_1x12_P2.54mm_Horizontal; moved to F.Cu
- J4, R1, R2, R6: moved to F.Cu
- J5: footprint Connector_USB:USB_C_Receptacle_Amphenol_12401548E4-2A -> Connector_USB:USB_C_Receptacle_GCT_USB4085; moved to B.Cu
- moved J2 63.1 mm to (38.7, 116.4), turned to 0 degrees
- moved R9 57.0 mm to (50.6, 151.8), turned to 180 degrees
- moved R10 55.3 mm to (50.6, 150.6), turned to 180 degrees
- moved C15 39.7 mm to (71.4, 89.9), turned to 0 degrees
- moved C18 36.0 mm to (77.4, 95.8), turned to 90 degrees
- moved U3 28.6 mm to (71.4, 97.0), turned to -90 degrees
- moved R7 16.3 mm to (57.2, 97.6), turned to 0 degrees
- moved SW1 16.1 mm to (52.9, 107.6)
- moved C1 15.5 mm to (46.4, 107.8), turned to -90 degrees
- moved SW2 15.5 mm to (45.7, 87.2)
- moved C2 15.5 mm to (46.4, 112.5), turned to -90 degrees
- moved J5 14.3 mm to (57.2, 95.1), turned to 0 degrees
- moved D9 14.1 mm to (70.8, 110.7)
- moved R1 12.2 mm to (50.0, 105.4)
- moved R2 11.9 mm to (50.0, 114.9)
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Connections:
- net GPIO25 renamed GPIO_25
- J2 pad 2: GPIO_19 -> +3V3
- J4 pad 2: /SWCLK -> /SWDIO
- J4 pad 3: /SWDIO -> /SWCLK
- U2 pad 11: Col 8 -> Col 5
- U2 pad 12: Col 9 -> Col 4
- U2 pad 13: Col 10 -> Col 3
- U2 pad 14: Col 11 -> Col 2
- U2 pad 15: Col 12 -> Col 1
- U2 pad 16: Col 13 -> Col 0
- U2 pad 17: Row 0 -> Row 4
- U2 pad 18: Row 1 -> Row 3
- U2 pad 2: Col 0 -> Col 13
- U2 pad 28: Row 3 -> Row 1
- U2 pad 29: Row 4 -> Row 0
- U2 pad 3: Col 1 -> Col 12
- U2 pad 30: GPIO_19 -> unconnected-(U2-Pad30)
- U2 pad 4: Col 2 -> Col 11
- U2 pad 5: Col 3 -> Col 10
- U2 pad 6: Col 4 -> Col 9
- U2 pad 7: Col 5 -> Col 8
- U2 pad 8: Col 6 -> Col 7
- U2 pad 9: Col 7 -> Col 6
Routing:
- net Col 7: track 131.9 -> 434.0 mm
- net Col 13: track 356.5 -> 500.7 mm
- net Col 12: track 359.5 -> 486.5 mm
- net Col 10: track 365.6 -> 476.1 mm
- net Col 11: track 390.2 -> 495.0 mm
- net USB_D+: track 2.39 -> 92.0 mm
- net USB_D-: track 2.39 -> 90.6 mm
- net Col 0: track 94.0 -> 170.0 mm
- net Col 6: track 316.9 -> 389.2 mm
- net Row 3: track 317.2 -> 367.4 mm, vias 0 -> 1
- net Col 4: track 201.5 -> 251.7 mm
- net Row 4: track 336.5 -> 376.0 mm, vias 0 -> 1
- net Col 5: track 235.9 -> 275.4 mm
- net Col 1: track 131.8 -> 170.2 mm
- net GPIO_22: track 0.00 -> 37.8 mm
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Other:
- board outline added: 363.5 x 98.8 mm

Commit message: PCB: All
Parts:
- D9: moved to F.Cu
- R6: moved to B.Cu
- moved SW2 43.1 mm to (57.5, 128.7), turned to 0 degrees
- moved D9 5.98 mm to (70.2, 116.7)
- moved U3 1.33 mm to (72.0, 98.2)
- moved C15 1.33 mm to (72.0, 91.1)
- moved C18 1.33 mm to (78.0, 97.0)
- moved R7 0.50 mm to (57.7, 97.6)
- moved C19 0.49 mm to (51.2, 149.6)
- moved C4 0.49 mm to (51.2, 148.4)
- moved R6 0.09 mm to (62.5, 91.7)
Routing:
- net Row 0: track 277.9 -> 343.8 mm, vias 0 -> 1
- net Row 4: track 376.0 -> 436.5 mm
- net Row 1: track 278.0 -> 325.2 mm, vias 0 -> 1
- net Row 2: track 331.8 -> 373.5 mm, vias 0 -> 1
- net GND: track 28.4 -> 65.3 mm, vias 8 -> 18
- net /VREG_VOUT: track 15.6 -> 36.7 mm, vias 2 -> 3
- net Net-(R5-Pad2): track 9.85 -> 28.7 mm, vias 0 -> 1
- net Col 0: track 170.0 -> 176.6 mm
- net VBUS: track 6.96 -> 12.0 mm
- net Net-(D9-Pad2): track 0.00 -> 3.86 mm
- net Net-(J5-PadA5): track 0.00 -> 2.74 mm
- net +3V3: track 41.2 -> 38.5 mm, vias 0 -> 2
- net Net-(J5-PadB5): track 0.00 -> 2.29 mm
- net Row 3: track 367.4 -> 366.4 mm
- net (no net): vias 1 -> 0
- added copper zone on F.Cu, net +3V3
- added copper zone on B.Cu, net GND
- added copper zone on F.Cu, net GND
- added copper zone on F.Cu, net VBUS

Commit message: PCB: Fix Errors
Parts:
- moved R6 4.17 mm to (66.7, 91.7), turned to -90 degrees
- moved J2 3.57 mm to (42.3, 116.4)
Routing:
- net Net-(C14-Pad2): track 14.8 -> 9.53 mm
- net Net-(J5-PadB5): track 2.29 -> 6.18 mm
- net GPIO_29: track 25.4 -> 21.9 mm
- net GPIO_28: track 27.0 -> 23.4 mm
- net GPIO_27: track 28.6 -> 25.0 mm
- net GPIO_26: track 30.1 -> 26.6 mm
- net GPIO_25: track 31.7 -> 28.2 mm
- net /XIN: track 18.7 -> 16.1 mm
- net GND: track 65.3 -> 62.8 mm
- net GPIO_24: track 33.2 -> 30.9 mm
- net GPIO_23: track 35.5 -> 33.6 mm
- net GPIO_22: track 37.8 -> 36.3 mm
- net Row 3: track 366.4 -> 365.8 mm
Other:
- board size 363.5 x 98.8 mm -> 363.1 x 99.4 mm

Commit message: Move all smd on one side
Parts:
- C10, C11, C12, C13, C14, C15, C16, C17, C18, C19, C3, C4, C5, C6, C7, C8, C9, D9, R1, R10, R2, R3, R4, R5, R8, R9, U1, U2, U3, Y1: moved to B.Cu
- J1: footprint Connector_PinHeader_2.54mm:PinHeader_1x02_P2.54mm_Vertical -> Button_Switch_SMD:SW_SPDT_PCM12
- J4: footprint Connector_PinHeader_2.54mm:PinHeader_1x04_P2.54mm_Horizontal -> Connector_PinSocket_2.54mm:PinSocket_1x04_P2.54mm_Horizontal
- J5: moved to F.Cu
- SW2: footprint Button_Switch_THT:SW_PUSH_6mm_H4.3mm -> Button_Switch_THT:SW_Tactile_SPST_Angled_PTS645Vx83-2LFS
- moved R3 43.6 mm to (75.0, 139.9), turned to 90 degrees
- moved R4 41.3 mm to (75.8, 142.3), turned to 180 degrees
- moved SW2 38.2 mm to (34.7, 159.4), turned to 90 degrees
- moved J4 38.2 mm to (41.9, 164.0), turned to 0 degrees
- moved C18 35.8 mm to (42.3, 95.3)
- moved C3 30.3 mm to (65.7, 140.1), turned to 0 degrees
- moved J1 28.1 mm to (33.9, 147.6), turned to -90 degrees
- moved U1 27.8 mm to (68.7, 144.8), turned to 180 degrees
- moved C15 23.9 mm to (48.2, 89.3), turned to 180 degrees
- moved U3 23.9 mm to (48.2, 96.4)
- moved R5 20.5 mm to (55.2, 167.5), turned to 45 degrees
- moved Y1 18.4 mm to (63.9, 172.2), turned to 0 degrees
- moved C14 16.0 mm to (62.2, 168.8), turned to 0 degrees
- moved C16 16.0 mm to (60.3, 166.9), turned to -90 degrees
- moved C10 15.9 mm to (51.8, 160.1), turned to 180 degrees
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Connections:
- C1 pad 1: GPIO 19 -> GPIO_28
- C2 pad 2: GPIO 20 -> GPIO_29
- J2 pad 10: GPIO_29 -> GND
- J2 pad 3: GPIO_22 -> GPIO_27
- J2 pad 4: GPIO_23 -> GPIO_26
- J2 pad 5: GPIO_24 -> GPIO_25
- J2 pad 6: GPIO_25 -> GPIO_24
- J2 pad 7: GPIO_26 -> GPIO_23
- J2 pad 8: GPIO_27 -> GPIO_22
- J2 pad 9: GPIO_28 -> GPIO_19
- R1 pad 1: GPIO 19 -> GPIO_28
- R2 pad 1: GPIO 20 -> GPIO_29
- SW1 pad A: GPIO 19 -> GPIO_28
- SW1 pad B: GPIO 20 -> GPIO_29
- U2 pad 11: Col 5 -> Col 6
- U2 pad 12: Col 4 -> Col 7
- U2 pad 13: Col 3 -> Col 8
- U2 pad 14: Col 2 -> Col 9
- U2 pad 15: Col 1 -> Col 10
- U2 pad 16: Col 0 -> Col 11
- U2 pad 17: Row 4 -> Col 12
- U2 pad 18: Row 3 -> Col 13
- U2 pad 2: Col 13 -> Row 0
- U2 pad 28: Row 1 -> Row 3
- U2 pad 29: Row 0 -> Row 4
- U2 pad 3: Col 12 -> Row 1
- U2 pad 30: unconnected-(U2-Pad30) -> GPIO_19
- U2 pad 4: Col 11 -> Col 0
- U2 pad 5: Col 10 -> Col 1
- U2 pad 6: Col 9 -> Col 2
- U2 pad 7: Col 8 -> Col 3
- U2 pad 8: Col 7 -> Col 4
- U2 pad 9: Col 6 -> Col 5
Routing:
- net Row 2: track 373.5 -> 434.9 mm, vias 1 -> 2
- net GPIO_19: track 0.00 -> 41.5 mm
- net Row 3: track 365.8 -> 406.5 mm, vias 1 -> 2
- net GPIO_28: track 23.4 -> 63.5 mm
- net Net-(R3-Pad2): track 5.39 -> 43.2 mm, vias 0 -> 1
- net OLED_SCL: track 11.6 -> 49.3 mm, vias 0 -> 2
- net OLED_SDA: track 12.5 -> 49.4 mm, vias 0 -> 2
- net GPIO_29: track 21.9 -> 55.6 mm
- net Row 4: track 436.5 -> 404.5 mm, vias 1 -> 2
- net USB_D+: track 92.0 -> 61.3 mm
- net USB_D-: track 90.6 -> 61.2 mm
- net Col 7: track 434.0 -> 404.7 mm, vias 0 -> 1
- net GPIO_27: track 25.0 -> 46.8 mm
- net GPIO_26: track 26.6 -> 44.8 mm
- net GPIO_25: track 28.2 -> 42.8 mm
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- removed copper zone on F.Cu, net +3V3
- removed copper zone on B.Cu, net GND
- removed copper zone on F.Cu, net GND
- removed copper zone on F.Cu, net VBUS
Other:
- outline, holes or cut-outs redrawn

Commit message: Rev 2 Draft
Routing:
- net Row 4: track 404.5 -> 475.7 mm, vias 2 -> 3
- net +3V3: track 39.5 -> 62.5 mm
- net GND: track 52.8 -> 56.9 mm, vias 17 -> 18
- net Col 1: track 165.4 -> 163.0 mm
- net VBUS: track 11.3 -> 13.1 mm
- net /VREG_VOUT: track 36.7 -> 38.4 mm, vias 3 -> 4
- net Col 0: track 169.4 -> 168.2 mm
- net Net-(R9-Pad1): track 5.47 -> 6.44 mm
- added copper zone on B.Cu, net +3V3
- added copper zone on B.Cu, net GND
- added copper zone on F.Cu, net GND
- added copper zone on B.Cu, net VBUS

Commit message: Cleanup
Routing:
- net Row 4: track 475.7 -> 474.6 mm
- net Row 3: track 406.5 -> 405.6 mm

Commit message: First prod rev
Parts:
- added REF**: MountingHole_2.2mm_M2_Pad_Via, MountingHole:MountingHole_2.2mm_M2_Pad_Via, F.Cu at (35.7, 181.0)
- added REF**: MountingHole_2.2mm_M2_Pad_Via, MountingHole:MountingHole_2.2mm_M2_Pad_Via, F.Cu at (184.5, 173.8)
- added REF**: MountingHole_2.2mm_M2_Pad_Via, MountingHole:MountingHole_2.2mm_M2_Pad_Via, F.Cu at (256.0, 173.8)
- added REF**: MountingHole_2.2mm_M2_Pad_Via, MountingHole:MountingHole_2.2mm_M2_Pad_Via, F.Cu at (231.0, 107.8)
- added REF**: MountingHole_2.2mm_M2_Pad_Via, MountingHole:MountingHole_2.2mm_M2_Pad_Via, F.Cu at (75.0, 92.3)
- added REF**: MountingHole_2.2mm_M2_Pad_Via, MountingHole:MountingHole_2.2mm_M2_Pad_Via, F.Cu at (350.6, 148.2)
- added REF**: MountingHole_2.2mm_M2_Pad_Via, MountingHole:MountingHole_2.2mm_M2_Pad_Via, F.Cu at (326.2, 107.8)
- added VBUS: TestPoint_THTPad_1.5x1.5mm_Drill0.7mm, TestPoint:TestPoint_THTPad_1.5x1.5mm_Drill0.7mm, F.Cu at (54.2, 97.0)
- moved J1 0.60 mm to (34.5, 147.6)
- moved R5 0.46 mm to (54.8, 167.3)
Routing:
- net +3V3: track 62.4 -> 48.0 mm
